Commit message: fix naming conventions, minor fixes to make the project run.

File: src/fishy_fish_navigation/urdf/mogi_bot.urdf (robot description, URDF)
Before this commit: robot mogi_bot, 10 links, 9 joints
Links:
- link base_link: geometry collision mesh filename=package://fishy_fish_navigation/meshes/base_link.STL; visual mesh filename=package://fishy_fish_navigation/meshes/base_link.STL
- link scan_link: geometry collision box size=.1 .1 .1; visual mesh filename=package://fishy_fish_navigation/meshes/lidar.dae
- link second_link: geometry collision mesh filename=package://fishy_fish_navigation/meshes/second_link.STL; visual mesh filename=package://fishy_fish_navigation/meshes/second_link.STL
- link tail_link: geometry collision mesh filename=package://fishy_fish_navigation/meshes/tail_link.STL; visual mesh filename=package://fishy_fish_navigation/meshes/tail_link.STL
- link third_link: geometry collision mesh filename=package://fishy_fish_navigation/meshes/third_link.STL; visual mesh filename=package://fishy_fish_navigation/meshes/third_link.STL
